Commit message: add visual, collision and inertial for wheels

File: src/rvc_robot_description/rvc_robot_description_common/urdf/components/wheel.urdf.xacro (robot description, xacro)
@@ -3,6 +3,20 @@
   <xacro:macro
     name="wheel"
-    params="prefix *origin parent:=base_link"
+    params="
+      prefix
+      *origin
+      parent:=base_link
+      config_file:='$(find rvc_robot_description_common)/config/wheel_params.yaml'
+    "
   >
+    <xacro:include filename="$(find rvc_robot_description_common)/urdf/utils/inertial_macros.xacro"/>
+    <xacro:property name="wheel_params" value="${xacro.load_yaml(config_file)}"/>
+    <!-- wheel geometric propreties -->
+    <xacro:property name="wheel_geometric" value="${wheel_params['geometric']}"/>
+    <xacro:property name="wheel_radius" value="${wheel_geometric['radius']}"/>
+    <xacro:property name="wheel_width" value="${wheel_geometric['width']}"/>
+    <!-- wheel physical propreties -->
+    <xacro:property name="wheel_physical" value="${wheel_params['physical']}"/>
+    <xacro:property name="wheel_mass" value="${wheel_physical['mass']}"/>
     <joint name="${prefix}_base_mount_joint" type="continuous">
       <xacro:insert_block name="origin"/>
@@ -11,5 +25,22 @@
       <axis xyz="0 1 0"/>
     </joint>
-    <link name="${prefix}_base_link"/>
+    <link name="${prefix}_base_link">
+      <visual>
+        <origin xyz="0 0 0" rpy="${pi/2} 0 0"/>
+        <geometry>
+          <cylinder radius="${wheel_radius}" length="${wheel_width}"/>
+        </geometry>
+      </visual>
+      <collision>
+        <origin xyz="0 0 0" rpy="${pi/2} 0 0"/>
+        <geometry>
+          <!-- use sphere to simplify friction -->
+          <sphere radius="${wheel_radius}"/>
+        </geometry>
+      </collision>
+      <xacro:inertial_cylinder mass="${wheel_mass}" radius="${wheel_radius}" length="${wheel_width}">
+        <origin xyz="0 0 0" rpy="${pi/2} 0 0"/>
+      </xacro:inertial_cylinder>
+    </link>
   </xacro:macro>
 </robot>

Commit message: separate wheel link and wheel base link

File: src/rvc_robot_description/rvc_robot_description_common/urdf/components/wheel.urdf.xacro (robot description, xacro)
@@ -19,11 +19,21 @@
     <xacro:property name="wheel_physical" value="${wheel_params['physical']}"/>
     <xacro:property name="wheel_mass" value="${wheel_physical['mass']}"/>
-    <joint name="${name}_base_mount_joint" type="continuous">
+    <joint name="${name}_base_mount_joint" type="fixed">
       <xacro:insert_block name="origin"/>
       <parent link="${parent}"/>
       <child link="${name}_base_link"/>
+    </joint>
+    <link name="${name}_base_link">
+      <xacro:inertial_cylinder mass="0.001" radius="0.001" length="0.01">
+        <origin xyz="0 0 0" rpy="0 0 0"/>
+      </xacro:inertial_cylinder>
+    </link>
+    <joint name="${name}_base_rotate_joint" type="continuous">
+      <origin xyz="0 0 0" rpy="0 0 0"/>
+      <parent link="${name}_base_link"/>
+      <child link="${name}"/>
       <axis xyz="0 1 0"/>
     </joint>
-    <link name="${name}_base_link">
+    <link name="${name}">
       <visual>
         <origin xyz="0 0 0" rpy="${pi/2} 0 0"/>
