Commit message: fix hardcoded caster wheel radius

File: src/rvc_robot_description/rvc_robot_description_common/urdf/components/caster_wheel.urdf.xacro (robot description, xacro)
@@ -29,5 +29,5 @@
       <visual>
         <geometry>
-          <sphere radius="0.006"/>
+          <sphere radius="${caster_wheel_mass}"/>
         </geometry>
         <material name="white"/>

Commit message: add materials.urdf.xacro

File: src/rvc_robot_description/rvc_robot_description_common/urdf/components/caster_wheel.urdf.xacro (robot description, xacro)
@@ -2,7 +2,4 @@
 <robot name="caster_wheel" xmlns:xacro="http://wiki.ros.org/xacro">
   <xacro:include filename="$(find rvc_robot_description_common)/urdf/utils/inertial_macros.xacro"/>
-  <material name="white">
-    <color rgba="1 1 1 1"/>
-  </material>
   <xacro:macro
     name="caster_wheel"

File: src/rvc_robot_description/rvc_robot_description_common/urdf/robot.urdf.xacro (robot description, xacro)
@@ -3,4 +3,5 @@
   <xacro:property name="chassis_radius" value="0.15"/>
   <xacro:property name="chassis_height" value="0.067"/>
+  <xacro:include filename="$(find rvc_robot_description_common)/urdf/utils/materials.urdf.xacro"/>
   <xacro:include filename="$(find rvc_robot_description_common)/urdf/components/wheel.urdf.xacro"/>
   <xacro:include filename="$(find rvc_robot_description_common)/urdf/components/caster_wheel.urdf.xacro"/>

Commit message: add collision and inertial for caster wheel

File: src/rvc_robot_description/rvc_robot_description_common/urdf/components/caster_wheel.urdf.xacro (robot description, xacro)
@@ -1,4 +1,5 @@
 <?xml version="1.0"?>
 <robot name="caster_wheel" xmlns:xacro="http://wiki.ros.org/xacro">
+  <xacro:include filename="$(find rvc_robot_description_common)/urdf/utils/inertial_macros.xacro"/>
   <material name="white">
     <color rgba="1 1 1 1"/>
@@ -6,6 +7,18 @@
   <xacro:macro
     name="caster_wheel"
-    params="prefix:=caster_wheel *origin parent:=base_link"
+    params="
+      prefix:=caster_wheel
+      *origin
+      parent:=base_link
+      config_file:='$(find rvc_robot_description_common)/config/caster_wheel_params.yaml'
+    "
   >
+    <xacro:property name="caster_wheel_params" value="${xacro.load_yaml(config_file)}"/>
+    <!-- caster wheel geometric propreties -->
+    <xacro:property name="caster_wheel_geometric" value="${caster_wheel_params['geometric']}"/>
+    <xacro:property name="caster_wheel_radius" value="${caster_wheel_geometric['radius']}"/>
+    <!-- caster wheel physical propreties -->
+    <xacro:property name="caster_wheel_physical" value="${caster_wheel_params['physical']}"/>
+    <xacro:property name="caster_wheel_mass" value="${caster_wheel_physical['mass']}"/>
     <joint name="${prefix}_base_mount_joint" type="fixed">
       <xacro:insert_block name="origin"/>
@@ -20,4 +33,14 @@
         <material name="white"/>
       </visual>
+      <collision>
+        <origin xyz="0 0 0" rpy="0 0 0"/>
+        <geometry>
+          <!-- use sphere to simplify friction -->
+          <sphere radius="${caster_wheel_radius}"/>
+        </geometry>
+      </collision>
+      <xacro:inertial_sphere mass="${caster_wheel_mass}" radius="${caster_wheel_radius}">
+        <origin xyz="0 0 0" rpy="0 0 0"/>
+      </xacro:inertial_sphere>
     </link>
   </xacro:macro>

Commit message: change xacro param "prefix" -> "name"

File: src/rvc_robot_description/rvc_robot_description_common/urdf/components/caster_wheel.urdf.xacro (robot description, xacro)
@@ -5,5 +5,5 @@
     name="caster_wheel"
     params="
-      prefix:=caster_wheel
+      name:=caster_wheel
       *origin
       parent:=base_link
@@ -18,10 +18,10 @@
     <xacro:property name="caster_wheel_physical" value="${caster_wheel_params['physical']}"/>
     <xacro:property name="caster_wheel_mass" value="${caster_wheel_physical['mass']}"/>
-    <joint name="${prefix}_base_mount_joint" type="fixed">
+    <joint name="${name}_base_mount_joint" type="fixed">
       <xacro:insert_block name="origin"/>
       <parent link="${parent}"/>
-      <child link="${prefix}_base_link"/>
+      <child link="${name}_base_link"/>
     </joint>
-    <link name="${prefix}_base_link">
+    <link name="${name}_base_link">
       <visual>
         <geometry>

File: src/rvc_robot_description/rvc_robot_description_common/urdf/components/chassis.urdf.xacro (robot description, xacro)
@@ -5,5 +5,5 @@
     name="chassis"
     params="
-      prefix
+      name
       *origin
       parent:=base_link
@@ -19,10 +19,10 @@
     <xacro:property name="chassis_physical" value="${chassis_params['physical']}"/>
     <xacro:property name="chassis_mass" value="${chassis_physical['mass']}"/>
-    <joint name="${prefix}_base_mount_joint" type="fixed">
+    <joint name="${name}_base_mount_joint" type="fixed">
       <xacro:insert_block name="origin"/>
       <parent link="${parent}"/>
-      <child link="${prefix}_base_link"/>
+      <child link="${name}_base_link"/>
     </joint>
-    <link name="${prefix}_base_link">
+    <link name="${name}_base_link">
       <visual>
         <origin xyz="0 0 0" rpy="0 0 0"/>

File: src/rvc_robot_description/rvc_robot_description_common/urdf/components/wheel.urdf.xacro (robot description, xacro)
@@ -4,5 +4,5 @@
     name="wheel"
     params="
-      prefix
+      name
       *origin
       parent:=base_link
@@ -19,11 +19,11 @@
     <xacro:property name="wheel_physical" value="${wheel_params['physical']}"/>
     <xacro:property name="wheel_mass" value="${wheel_physical['mass']}"/>
-    <joint name="${prefix}_base_mount_joint" type="continuous">
+    <joint name="${name}_base_mount_joint" type="continuous">
       <xacro:insert_block name="origin"/>
       <parent link="${parent}"/>
-      <child link="${prefix}_base_link"/>
+      <child link="${name}_base_link"/>
       <axis xyz="0 1 0"/>
     </joint>
-    <link name="${prefix}_base_link">
+    <link name="${name}_base_link">
       <visual>
         <origin xyz="0 0 0" rpy="${pi/2} 0 0"/>

File: src/rvc_robot_description/rvc_robot_description_common/urdf/robot.urdf.xacro (robot description, xacro)
@@ -18,15 +18,15 @@
   </link>
   <xacro:chassis
-    prefix="chassis"
+    name="chassis"
   >
     <origin xyz="0 0 ${chassis_height/2}" rpy="0 0 0"/>
   </xacro:chassis>
   <xacro:wheel
-    prefix="left_wheel"
+    name="left_wheel"
   >
     <origin xyz="0 ${chassis_radius} 0" rpy="0 0 0"/>
   </xacro:wheel>
   <xacro:wheel
-    prefix="right_wheel"
+    name="right_wheel"
   >
     <origin xyz="0 -${chassis_radius} 0" rpy="0 0 0"/>

Commit message: separate caster base_link and caster link

File: src/rvc_robot_description/rvc_robot_description_common/urdf/components/caster_wheel.urdf.xacro (robot description, xacro)
@@ -23,5 +23,11 @@
       <child link="${name}_base_link"/>
     </joint>
-    <link name="${name}_base_link">
+    <link name="${name}_base_link"/>
+    <joint name="${name}_base_fixed_joint" type="fixed">
+      <origin xyz="0 0 -0.028" rpy="0 0 0"/>
+      <parent link="${name}_base_link"/>
+      <child link="${name}"/>
+    </joint>
+    <link name="${name}">
       <visual>
         <geometry>
