Commit message: add chassis

File: src/rvc_robot_description/rvc_robot_description_common/urdf/robot.urdf.xacro (robot description, xacro)
@@ -4,7 +4,13 @@
   <xacro:property name="chassis_height" value="0.067"/>
   <xacro:include filename="$(find rvc_robot_description_common)/urdf/utils/materials.urdf.xacro"/>
+  <xacro:include filename="$(find rvc_robot_description_common)/urdf/components/chassis.urdf.xacro"/>
   <xacro:include filename="$(find rvc_robot_description_common)/urdf/components/wheel.urdf.xacro"/>
   <xacro:include filename="$(find rvc_robot_description_common)/urdf/components/caster_wheel.urdf.xacro"/>
   <link name="base_link"/>
+  <xacro:chassis
+    prefix="chassis"
+  >
+    <origin xyz="0 0 ${chassis_height/2}" rpy="0 0 0"/>
+  </xacro:chassis>
   <xacro:wheel
     prefix="left_wheel"

Commit message: use chassis_params.yaml in main robot urdf file

File: src/rvc_robot_description/rvc_robot_description_common/urdf/robot.urdf.xacro (robot description, xacro)
@@ -1,6 +1,10 @@
 <?xml version="1.0"?>
 <robot name="rvc_common" xmlns:xacro="http://wiki.ros.org/xacro">
-  <xacro:property name="chassis_radius" value="0.15"/>
-  <xacro:property name="chassis_height" value="0.067"/>
+  <xacro:arg name="chassis_config_file" default="$(find rvc_robot_description_common)/config/chassis_params.yaml"/>
+  <xacro:property name="chassis_params" value="${xacro.load_yaml('$(arg chassis_config_file)')}"/>
+  <!-- chassis geometric propreties -->
+  <xacro:property name="chassis_geometric" value="${chassis_params['geometric']}"/>
+  <xacro:property name="chassis_radius" value="${chassis_geometric['radius']}"/>
+  <xacro:property name="chassis_height" value="${chassis_geometric['height']}"/>
   <xacro:include filename="$(find rvc_robot_description_common)/urdf/utils/materials.urdf.xacro"/>
   <xacro:include filename="$(find rvc_robot_description_common)/urdf/components/chassis.urdf.xacro"/>

Commit message: add dummy inertial to satisfy gazebo

File: src/rvc_robot_description/rvc_robot_description_common/urdf/robot.urdf.xacro (robot description, xacro)
@@ -8,8 +8,13 @@
   <xacro:property name="chassis_height" value="${chassis_geometric['height']}"/>
   <xacro:include filename="$(find rvc_robot_description_common)/urdf/utils/materials.urdf.xacro"/>
+  <xacro:include filename="$(find rvc_robot_description_common)/urdf/utils/inertial_macros.xacro"/>
   <xacro:include filename="$(find rvc_robot_description_common)/urdf/components/chassis.urdf.xacro"/>
   <xacro:include filename="$(find rvc_robot_description_common)/urdf/components/wheel.urdf.xacro"/>
   <xacro:include filename="$(find rvc_robot_description_common)/urdf/components/caster_wheel.urdf.xacro"/>
-  <link name="base_link"/>
+  <link name="base_link">
+    <xacro:inertial_cylinder mass="0.001" radius="0.001" length="0.01">
+      <origin xyz="0 0 0" rpy="0 0 0"/>
+    </xacro:inertial_cylinder>
+  </link>
   <xacro:chassis
     prefix="chassis"
